File: Ai3MS_connector_board.sch (KiCad schematic (older format))
At the start: 10 parts, among them J1 2x7, T0 1x2

Commit message: Add EXTRUDER and BLTOUCH
Parts:
- added BLTOUCH1: 1x5, Connector_JST:JST_XH_B5B-XH-A_1x05_P2.50mm_Vertical, symbol mogira:1x5
- added EXTRUDER1: 1x4, Connector_JST:JST_XH_B4B-XH-A_1x04_P2.50mm_Vertical, symbol mogira:1x4
- added J2: 1x4_rev, Connector_JST:JST_XH_B4B-XH-A_1x04_P2.50mm_Vertical, symbol mogira:1x4_rev
- added J3: 1x3_rev, Connector_JST:JST_XH_B3B-XH-A_1x03_P2.50mm_Vertical, symbol mogira:1x3_rev
Connections:
- net P5 renamed BLTOUCH1_WHITE
- net BLTOUCH1_WHITE: now also BLTOUCH1.2 (Pin_2)
- net T0_P2 renamed BLTOUCH1_BLUE
- net BLTOUCH1_BLUE: now also BLTOUCH1.1 (Pin_1)
- new net: EXTRUDER1.1 (Pin_1), J2.1 (Pin_1)
- new net: EXTRUDER1.2 (Pin_2), J2.2 (Pin_2)
- new net: EXTRUDER1.3 (Pin_3), J2.3 (Pin_3)
- new net: EXTRUDER1.4 (Pin_4), J2.4 (Pin_4)
- new net BLTOUCH1_BROWN: BLTOUCH1.4 (Pin_4), J3.2 (Pin_2)
- new net BLTOUCH1_RED: BLTOUCH1.5 (Pin_5), J3.3 (Pin_3)
- new net BLTOUCH1_YELLOW: BLTOUCH1.3 (Pin_3), J3.1 (Pin_1)
Changed lines of the file:
@@
 EESchema Schematic File Version 4
+LIBS:Ai3MS_connector_board-cache
 EELAYER 29 0
 EELAYER END
@@
 Wire Wire Line
 	3200 4500 3350 4500
+Wire Wire Line
+	2150 4400 2250 4400
 Text GLabel 2150 4400 0    50   Input ~ 0
 P5
@@
 Wire Wire Line
 	3200 4300 3350 4300
+Wire Wire Line
+	3350 4500 3450 4500
 Text GLabel 3550 4500 2    50   Input ~ 0
 T0_P2
@@
 	1    0    0    -1
 $EndComp
-Wire Wire Line
-	3350 4500 3550 4500
-Wire Wire Line
-	2150 4400 2900 4400
+$Comp
+L mogira:1x4_rev J2
+U 1 1 5F1321D5
+P 4400 2450
+F 0 "J2" H 4400 2200 50  0000 C CNN
+F 1 "1x4_rev" H 4550 2500 25  0001 C CNN
+F 2 "Connector_JST:JST_XH_B4B-XH-A_1x04_P2.50mm_Vertical" H 4400 2500 50  0001 C CNN
+F 3 "" H 4400 2500 50  0001 C CNN
+	1    4400 2450
+	1    0    0    -1
+$EndComp
+Wire Wire Line
+	3450 4500 3450 4650
+Wire Wire Line
+	3450 4650 3550 4650
+Connection ~ 3450 4500
+Wire Wire Line
+	3450 4500 3550 4500
+Text GLabel 3550 4650 2    50   Input ~ 0
+BLTOUCH1_BLUE
+Text GLabel 2150 4550 0    50   Input ~ 0
+BLTOUCH1_WHITE
+Wire Wire Line
+	2150 4550 2250 4550
+Wire Wire Line
+	2250 4550 2250 4400
+Connection ~ 2250 4400
+Wire Wire Line
+	2250 4400 2900 4400
+Text GLabel 6725 2300 0    50   Input ~ 0
+BLTOUCH1_BLUE
+Wire Wire Line
+	6725 2300 6950 2450
+Text GLabel 6750 2450 0    50   Input ~ 0
+BLTOUCH1_WHITE
+Wire Wire Line
+	6750 2450 6950 2550
+Text Label 6100 2650 0    50   ~ 0
+BLTOUCH1_YELLOW
+Text Label 6150 2850 0    50   ~ 0
+BLTOUCH1_RED
+Text Label 6100 2750 0    50   ~ 0
+BLTOUCH1_BROWN
+$Comp
+L mogira:1x5 BLTOUCH1
+U 1 1 5F179B7D
+P 7050 2650
+F 0 "BLTOUCH1" H 7128 2650 50  0000 L CNN
+F 1 "1x5" H 7128 2604 25  0001 L CNN
+F 2 "Connector_JST:JST_XH_B5B-XH-A_1x05_P2.50mm_Vertical" H 7050 2700 50  0001 C CNN
+F 3 "" H 7050 2700 50  0001 C CNN
+	1    7050 2650
+	1    0    0    -1
+$EndComp
+$Comp
+L mogira:1x3_rev J3
+U 1 1 5F1884C2
+P 5850 2750
+F 0 "J3" H 5850 2550 50  0000 C CNN
+F 1 "1x3_rev" H 5883 2953 25  0001 C CNN
+F 2 "Connector_JST:JST_XH_B3B-XH-A_1x03_P2.50mm_Vertical" H 5850 2800 50  0001 C CNN
+F 3 "" H 5850 2800 50  0001 C CNN
+	1    5850 2750
+	1    0    0    -1
+$EndComp
+Wire Wire Line
+	6950 2650 5950 2650
+Wire Wire Line
+	6950 2750 5950 2750
+Wire Wire Line
+	5950 2850 6950 2850
+Wire Wire Line
+	4750 2600 4500 2600
+Wire Wire Line
+	4500 2500 4750 2500
+Wire Wire Line
+	4750 2400 4500 2400
+Wire Wire Line
+	4500 2300 4750 2300
+$Comp
+L mogira:1x4 EXTRUDER1
+U 1 1 5F12BC10
+P 4850 2450
+F 0 "EXTRUDER1" H 4928 2450 50  0000 L CNN
+F 1 "1x4" H 4928 2404 25  0001 L CNN
+F 2 "Connector_JST:JST_XH_B4B-XH-A_1x04_P2.50mm_Vertical" H 4850 2500 50  0001 C CNN
+F 3 "" H 4850 2500 50  0001 C CNN
+	1    4850 2450
+	1    0    0    -1
+$EndComp
 $EndSCHEMATC

Commit message: Remove SWITCH, Capacitors and Resistors
Parts:
- removed C1: 1uF, Capacitor_SMD:C_0603_1608Metric_Pad1.05x0.95mm_HandSolder, symbol Device:C_Small
- removed C2: 100NF, Capacitor_SMD:C_0603_1608Metric_Pad1.05x0.95mm_HandSolder, symbol Device:C_Small
- removed R1: 15K, Resistor_SMD:R_0603_1608Metric_Pad1.05x0.95mm_HandSolder, symbol Device:R_Small
- removed R2: 10K, Resistor_SMD:R_0603_1608Metric_Pad1.05x0.95mm_HandSolder, symbol Device:R_Small
- removed SWITCH1: SW_SPDT, Button_Switch_THT:SW_CuK_OS102011MA1QN1_SPDT_Angled, symbol Switch:SW_SPDT
Changed lines of the file:
@@
 	3200 4500 3350 4500
-Wire Wire Line
-	2150 4400 2250 4400
-Text GLabel 2150 4400 0    50   Input ~ 0
-P5
 Wire Wire Line
 	3200 4600 3250 4600
@@
 Text GLabel 2550 4200 0    50   Input ~ 0
 HOTEND1_P1
-Wire Wire Line
-	6200 4200 6150 4200
-$Comp
-L Device:R_Small R1
-U 1 1 5F124A70
-P 6350 4000
-F 0 "R1" V 6550 3950 50  0001 L CNN
-F 1 "15K" V 6450 3900 50  0000 L CNN
-F 2 "Resistor_SMD:R_0603_1608Metric_Pad1.05x0.95mm_HandSolder" H 6350 4000 50  0001 C CNN
-F 3 "~" H 6350 4000 50  0001 C CNN
-	1    6350 4000
-	0    -1   -1   0
-$EndComp
-Wire Wire Line
-	6150 4000 6250 4000
-Text GLabel 7350 4000 2    50   Input ~ 0
-P5
-$Comp
-L Device:R_Small R2
-U 1 1 5F12F25C
-P 6600 4200
-F 0 "R2" H 6659 4246 50  0001 L CNN
-F 1 "10K" H 6659 4155 50  0000 L CNN
-F 2 "Resistor_SMD:R_0603_1608Metric_Pad1.05x0.95mm_HandSolder" H 6600 4200 50  0001 C CNN
-F 3 "~" H 6600 4200 50  0001 C CNN
-	1    6600 4200
-	1    0    0    -1
-$EndComp
-$Comp
-L Device:C_Small C2
-U 1 1 5F12F262
-P 6950 4200
-F 0 "C2" H 7042 4246 50  0001 L CNN
-F 1 "100NF" H 7042 4155 50  0000 L CNN
-F 2 "Capacitor_SMD:C_0603_1608Metric_Pad1.05x0.95mm_HandSolder" H 6950 4200 50  0001 C CNN
-F 3 "~" H 6950 4200 50  0001 C CNN
-	1    6950 4200
-	1    0    0    -1
-$EndComp
-Wire Wire Line
-	6950 4300 6950 4400
-Wire Wire Line
-	6600 4100 6600 4000
-Wire Wire Line
-	6600 4300 6600 4400
-Connection ~ 6600 4000
-Connection ~ 6600 4400
-Wire Wire Line
-	6950 4000 6950 4100
-Wire Wire Line
-	6950 4000 7350 4000
-$Comp
-L Switch:SW_SPDT SWITCH1
-U 1 1 5F11AF04
-P 5950 4100
-F 0 "SWITCH1" H 5950 4293 50  0000 C CNN
-F 1 "SW_SPDT" H 5950 4294 50  0001 C CNN
-F 2 "Button_Switch_THT:SW_CuK_OS102011MA1QN1_SPDT_Angled" H 5950 4100 50  0001 C CNN
-F 3 "~" H 5950 4100 50  0001 C CNN
-	1    5950 4100
-	1    0    0    -1
-$EndComp
-Wire Wire Line
-	6200 4200 6200 4400
-Text GLabel 5550 3850 0    50   Input ~ 0
-FAN0_P1
-Text GLabel 5450 4000 0    50   Input ~ 0
-FAN2_P1
-Wire Wire Line
-	5200 4350 5200 4400
-Wire Wire Line
-	5200 4400 6200 4400
-Text GLabel 7300 4400 2    50   Input ~ 0
-T0_P2
-Wire Wire Line
-	6950 4400 7300 4400
-Wire Wire Line
-	5550 3850 5650 3850
-Wire Wire Line
-	5450 4000 5550 4000
-Wire Wire Line
-	5550 4000 5550 4100
-Wire Wire Line
-	5550 4100 5650 4100
-Wire Wire Line
-	5650 3850 5650 4100
-Wire Wire Line
-	5650 4100 5750 4100
-Connection ~ 5650 4100
-$Comp
-L Device:C_Small C1
-U 1 1 5F11BFAD
-P 5200 4250
-F 0 "C1" H 5000 4300 50  0001 L CNN
-F 1 "1uF" H 4950 4250 50  0000 L CNN
-F 2 "Capacitor_SMD:C_0603_1608Metric_Pad1.05x0.95mm_HandSolder" H 5200 4250 50  0001 C CNN
-F 3 "~" H 5200 4250 50  0001 C CNN
-	1    5200 4250
-	1    0    0    -1
-$EndComp
-Connection ~ 5550 4100
-Wire Wire Line
-	5200 4100 5200 4150
-Wire Wire Line
-	5200 4100 5550 4100
-Wire Wire Line
-	6600 4000 6950 4000
-Connection ~ 6950 4000
-Wire Wire Line
-	6450 4000 6600 4000
-Wire Wire Line
-	6200 4400 6600 4400
-Connection ~ 6200 4400
-Wire Wire Line
-	6600 4400 6950 4400
-Connection ~ 6950 4400
 Connection ~ 3350 4500
 Wire Wire Line
@@
 Text GLabel 3550 4650 2    50   Input ~ 0
 BLTOUCH1_BLUE
-Text GLabel 2150 4550 0    50   Input ~ 0
+Text GLabel 2700 4400 0    50   Input ~ 0
 BLTOUCH1_WHITE
-Wire Wire Line
-	2150 4550 2250 4550
-Wire Wire Line
-	2250 4550 2250 4400
-Connection ~ 2250 4400
-Wire Wire Line
-	2250 4400 2900 4400
 Text GLabel 6725 2300 0    50   Input ~ 0
 BLTOUCH1_BLUE
@@
 	1    0    0    -1
 $EndComp
+Wire Wire Line
+	3550 3550 3450 3550
+Text GLabel 3550 3550 2    50   Input ~ 0
+FAN0_P1
+Wire Wire Line
+	3450 3550 3450 3700
+Connection ~ 3450 3700
+Wire Wire Line
+	2900 4400 2700 4400
 $EndSCHEMATC
