File: pcb/Ai3MS_connector_board.kicad_pcb (KiCad board)
At the start: 2 copper layers, 47 x 22.1 mm, 11 parts

Commit message: Export symbols and footprints to libraries
Parts:
- MainConnector: footprint mogira:PHLike_Green_Connector -> Ai3MS_connector_board:PHLike_Green_Connector
- REF** (x2): footprint mogira:AXA-15-M3 -> Ai3MS_connector_board:AXA-15-M3
Changed lines of the file:
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@@
     )
   )
-  (module mogira:AXA-15-M3 (layer B.Cu)
+  (module Ai3MS_connector_board:AXA-15-M3 (layer B.Cu)
     (at 174.63 117.285)
     (fp_text reference REF** (at 0 -2.53) (layer B.SilkS) hide
@@
     (pad 1 thru_hole circle (at 0 0) (size 3 3) (drill 1.6) (layers *.Cu *.Mask))
   )
-  (module mogira:AXA-15-M3 (layer B.Cu)
+  (module Ai3MS_connector_board:AXA-15-M3 (layer B.Cu)
     (at 138.78 117.285)
     (fp_text reference REF** (at 0 -2.53) (layer B.SilkS) hide
@@
     )
   )
-  (module mogira:PHLike_Green_Connector (layer F.Cu)
+  (module Ai3MS_connector_board:PHLike_Green_Connector (layer F.Cu)
     (at 153.63 109.76 270)
     (descr "2mm pitch green connector used in Anycubic i3 Mega")
