File: pcb/Ai3MS_connector_board.kicad_pcb (KiCad board)
At the start: 2 copper layers, 47 x 22.1 mm, 11 parts

Commit message: Improve links
* Change link names
* Change connection paths
* Retouch PCB due to loading new net file

* Note: HEATER's 12V/GND is inversed of others. Pin#1 is GND, Pin#2 is 12V.
Parts:
- renumbered BLTOUCH to BLTouch, EXTRUDER to Extruder, MainConnector to J1
Connections:
- net /BLTOUCH1_BROWN renamed /BLTOUCH1_SERVO_GND
- net /BLTOUCH1_RED renamed /BLTOUCH1_SERVO_5V
- net /BLTOUCH1_YELLOW renamed /BLTOUCH1_SERVO_CONTROL
- net BLTOUCH1_BLUE renamed BLTOUCH1_GND
- net BLTOUCH1_WHITE renamed BLTOUCH1_ZMIN
- net FAN0_P1 renamed HEATER1_12V
- net FAN0_P2 renamed PARTFAN1_GND
- net FAN2_P2 renamed HOTENDFAN1_GND
- net HOTEND1_P1 renamed HEATER1_GND
- net Net-(EXTRUDER1-Pad1) renamed /EXTRUDER1_A+
- net Net-(EXTRUDER1-Pad2) renamed /EXTRUDER1_A-
- net Net-(EXTRUDER1-Pad3) renamed /EXTRUDER1_B+
- net Net-(EXTRUDER1-Pad4) renamed /EXTRUDER1_B-
- net T0_P1 renamed THERMISTOR1_DATA
