File: pcb/Ai3MS_connector_board.kicad_pcb (KiCad board)
At the start: 2 copper layers, 47 x 22.1 mm, 11 parts, among them J1 2x7

Commit message: Improve 2x7_2mm-pitch_Lock_GreenConnector
* Renamed from "PHLike_Green_Connector"
* Fix pin assign of symbol "2x7"
* Fix pin assign of footprint "2x7_2mm-pitch_Lock_GreenConnector"
* Update silk
* Add 3d model
Parts:
- J1: footprint Ai3MS_connector_board:PHLike_Green_Connector -> Ai3MS_connector_board:2x7_2mm-pitch_Lock_GreenConnector
Connections:
- J1 pad 11: PARTFAN1_GND -> BLTOUCH1_GND
- J1 pad 12: HOTENDFAN1_GND -> BLTOUCH1_GND
- J1 pad 13: HEATER1_GND -> THERMISTOR1_DATA
- J1 pad 14: HEATER1_12V -> THERMISTOR1_DATA
- J1 pad 3: HEATER1_GND -> HEATER1_12V
- J1 pad 5: BLTOUCH1_ZMIN -> HEATER1_GND
- J1 pad 6: BLTOUCH1_GND -> HOTENDFAN1_GND
- J1 pad 7: THERMISTOR1_DATA -> HEATER1_GND
- J1 pad 8: THERMISTOR1_DATA -> PARTFAN1_GND
- J1 pad 9: BLTOUCH1_GND -> BLTOUCH1_ZMIN
Changed lines of the file:
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@@
     (uvia_drill 0.1)
+  )
+  (module Ai3MS_connector_board:2x7_2mm-pitch_Lock_GreenConnector (layer F.Cu)
+    (at 153.63 109.76 270)
+    (descr "2mm pitch green connector used in Anycubic i3 Mega")
+    (fp_text reference J1 (at 5.885 -1.75 90) (layer F.SilkS) hide
+      (effects (font (size 1 1) (thickness 0.15)))
+    )
+    (fp_text value 2x7 (at 6.155 -4.435 90) (layer F.Fab) hide
+      (effects (font (size 1 1) (thickness 0.15)))
+    )
+    (fp_text user 2 (at -1.4 2 90) (layer F.SilkS)
+      (effects (font (size 1 1) (thickness 0.15)))
+    )
+    (fp_text user 1 (at -1.4 0 90) (layer F.SilkS)
+      (effects (font (size 1 1) (thickness 0.15)))
+    )
+    (fp_line (start -2 3.8) (end 14 3.8) (layer F.SilkS) (width 0.12))
+    (fp_line (start 10.5 -3.3) (end 10.5 -2.6) (layer F.SilkS) (width 0.12))
+    (fp_line (start 1.5 -3.3) (end 1.5 -2.6) (layer F.SilkS) (width 0.12))
+    (fp_line (start 1.5 -3.3) (end 10.5 -3.3) (layer F.SilkS) (width 0.12))
+    (fp_line (start -2 4.6) (end 14 4.6) (layer F.SilkS) (width 0.12))
+    (fp_line (start -2 -2.6) (end 14 -2.6) (layer F.SilkS) (width 0.12))
+    (fp_line (start 14 -2.6) (end 14 4.6) (layer F.SilkS) (width 0.12))
+    (fp_line (start -2 -2.6) (end -2 4.6) (layer F.SilkS) (width 0.12))
+    (pad 2 thru_hole oval (at 0 2 270) (size 1.2 1.7) (drill 0.75) (layers *.Cu *.Mask)
+      (net 11 HEATER1_12V))
+    (pad 4 thru_hole oval (at 2 2 270) (size 1.2 1.7) (drill 0.75) (layers *.Cu *.Mask)
+      (net 12 HEATER1_GND))
+    (pad 6 thru_hole oval (at 4 2 270) (size 1.2 1.7) (drill 0.75) (layers *.Cu *.Mask)
+      (net 13 HOTENDFAN1_GND))
+    (pad 8 thru_hole oval (at 6 2 270) (size 1.2 1.7) (drill 0.75) (layers *.Cu *.Mask)
+      (net 14 PARTFAN1_GND))
+    (pad 10 thru_hole oval (at 8 2 270) (size 1.2 1.7) (drill 0.75) (layers *.Cu *.Mask)
+      (net 1 "Net-(J1-Pad10)"))
+    (pad 12 thru_hole oval (at 10 2 270) (size 1.2 1.7) (drill 0.75) (layers *.Cu *.Mask)
+      (net 2 BLTOUCH1_GND))
+    (pad 14 thru_hole oval (at 12 2 270) (size 1.2 1.7) (drill 0.75) (layers *.Cu *.Mask)
+      (net 15 THERMISTOR1_DATA))
+    (pad 13 thru_hole oval (at 12 0 270) (size 1.2 1.7) (drill 0.75) (layers *.Cu *.Mask)
+      (net 15 THERMISTOR1_DATA))
+    (pad 11 thru_hole oval (at 10 0 270) (size 1.2 1.7) (drill 0.75) (layers *.Cu *.Mask)
+      (net 2 BLTOUCH1_GND))
+    (pad 9 thru_hole oval (at 8 0 270) (size 1.2 1.7) (drill 0.75) (layers *.Cu *.Mask)
+      (net 3 BLTOUCH1_ZMIN))
+    (pad 7 thru_hole oval (at 6 0 270) (size 1.2 1.7) (drill 0.75) (layers *.Cu *.Mask)
+      (net 12 HEATER1_GND))
+    (pad 5 thru_hole oval (at 4 0 270) (size 1.2 1.7) (drill 0.75) (layers *.Cu *.Mask)
+      (net 12 HEATER1_GND))
+    (pad 3 thru_hole oval (at 2 0 270) (size 1.2 1.7) (drill 0.75) (layers *.Cu *.Mask)
+      (net 11 HEATER1_12V))
+    (pad 1 thru_hole rect (at 0 0 270) (size 1.2 1.7) (drill 0.75) (layers *.Cu *.Mask)
+      (net 11 HEATER1_12V))
+    (model ${KIPRJMOD}/libraries/Ai3MS_connector_board.pretty/2x7_2mm-pitch_Lock_GreenConnector.step
+      (at (xyz 0 0 0))
+      (scale (xyz 1 1 1))
+      (rotate (xyz 0 0 0))
+    )
   )
   (module Ai3MS_connector_board:AXA-15-M3 (layer B.Cu)
@@
     )
   )
-  (module Ai3MS_connector_board:PHLike_Green_Connector (layer F.Cu)
-    (at 153.63 109.76 270)
-    (descr "2mm pitch green connector used in Anycubic i3 Mega")
-    (fp_text reference J1 (at 6 5.425 90) (layer F.SilkS) hide
-      (effects (font (size 1 1) (thickness 0.15)))
-    )
-    (fp_text value 2x7 (at 5.99 5.295 90) (layer F.Fab) hide
-      (effects (font (size 1 1) (thickness 0.15)))
-    )
-    (fp_line (start 10.7 -3.0125) (end 10.7 -2.5) (layer F.SilkS) (width 1))
-    (fp_line (start 1.285 -3.005) (end 1.285 -2.515) (layer F.SilkS) (width 1))
-    (fp_line (start 1.3 -3.0125) (end 10.7 -3.0125) (layer F.SilkS) (width 1))
-    (fp_line (start -1.825 -2.25) (end 13.825 -2.25) (layer F.SilkS) (width 0.55))
-    (fp_line (start 13.825 -2.15) (end 13.825 4.15) (layer F.SilkS) (width 0.75))
-    (fp_line (start -1.825 4.25) (end 13.825 4.25) (layer F.SilkS) (width 0.55))
-    (fp_line (start -1.825 -2.15) (end -1.825 4.15) (layer F.SilkS) (width 0.75))
-    (pad 14 thru_hole oval (at 0 2 270) (size 1.2 1.7) (drill 0.75) (layers *.Cu *.Mask)
-      (net 11 HEATER1_12V))
-    (pad 13 thru_hole oval (at 2 2 270) (size 1.2 1.7) (drill 0.75) (layers *.Cu *.Mask)
-      (net 12 HEATER1_GND))
-    (pad 12 thru_hole oval (at 4 2 270) (size 1.2 1.7) (drill 0.75) (layers *.Cu *.Mask)
-      (net 13 HOTENDFAN1_GND))
-    (pad 11 thru_hole oval (at 6 2 270) (size 1.2 1.7) (drill 0.75) (layers *.Cu *.Mask)
-      (net 14 PARTFAN1_GND))
-    (pad 10 thru_hole oval (at 8 2 270) (size 1.2 1.7) (drill 0.75) (layers *.Cu *.Mask)
-      (net 1 "Net-(J1-Pad10)"))
-    (pad 9 thru_hole oval (at 10 2 270) (size 1.2 1.7) (drill 0.75) (layers *.Cu *.Mask)
-      (net 2 BLTOUCH1_GND))
-    (pad 8 thru_hole oval (at 12 2 270) (size 1.2 1.7) (drill 0.75) (layers *.Cu *.Mask)
-      (net 15 THERMISTOR1_DATA))
-    (pad 7 thru_hole oval (at 12 0 270) (size 1.2 1.7) (drill 0.75) (layers *.Cu *.Mask)
-      (net 15 THERMISTOR1_DATA))
-    (pad 6 thru_hole oval (at 10 0 270) (size 1.2 1.7) (drill 0.75) (layers *.Cu *.Mask)
-      (net 2 BLTOUCH1_GND))
-    (pad 5 thru_hole oval (at 8 0 270) (size 1.2 1.7) (drill 0.75) (layers *.Cu *.Mask)
-      (net 3 BLTOUCH1_ZMIN))
-    (pad 4 thru_hole oval (at 6 0 270) (size 1.2 1.7) (drill 0.75) (layers *.Cu *.Mask)
-      (net 12 HEATER1_GND))
-    (pad 3 thru_hole oval (at 4 0 270) (size 1.2 1.7) (drill 0.75) (layers *.Cu *.Mask)
-      (net 12 HEATER1_GND))
-    (pad 2 thru_hole oval (at 2 0 270) (size 1.2 1.7) (drill 0.75) (layers *.Cu *.Mask)
-      (net 11 HEATER1_12V))
-    (pad 1 thru_hole rect (at 0 0 270) (size 1.2 1.7) (drill 0.75) (layers *.Cu *.Mask)
-      (net 11 HEATER1_12V))
-  )
   (module Connector_JST:JST_PH_B2B-PH-K_1x02_P2.00mm_Vertical (layer B.Cu)

Commit message: Fix upper right silk
* From "ANYCUBIC i3 Mega" to "ANYCUBIC i3 Mega S"
* Update version string
Other:
- board text added: "ANYCUBIC i3 Mega S Connector Board for Direct Extruder with BLTouch ver 1.0.1"
- board text removed: "ANYCUBIC i3 Mega Connector Board for Direct Extruder with BLTouch ver 1.0.0"
Changed lines of the file:
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@@
     (effects (font (size 0.8 0.8) (thickness 0.14)))
   )
-  (gr_text "ANYCUBIC i3 Mega\nConnector Board\nfor Direct Extruder\nwith BLTouch\nver 1.0.0" (at 173.24 110.79) (layer F.SilkS)
+  (gr_text "ANYCUBIC i3 Mega S\nConnector Board\nfor Direct Extruder\nwith BLTouch\nver 1.0.1" (at 173.24 110.79) (layer F.SilkS)
     (effects (font (size 0.8 0.8) (thickness 0.14)))
   )
